File: Hardware/SparkFun_Artemis.sch (EAGLE design)
At the start: 68 parts, among them J1 PAD, J10 PAD, J11 PAD, J12 PAD, J13 PAD, J14 PAD, J15 PAD, J16 PAD, J17 PAD, J18 PAD, J19 PAD, J2 PAD, J20 PAD, J21 PAD, J22 PAD, J23 PAD, J24 PAD, J25 PAD, J26 PAD, J27 PAD, J28 PAD, J29 PAD, J3 PAD, J30 PAD, J31 PAD, J32 PAD, J33 PAD, J34 PAD, J35 PAD, J36 PAD, J37 PAD, J38 PAD, J39 PAD, J4 PAD, J40 PAD, J41 PAD, J42 PAD, J43 PAD, J5 PAD, J6 PAD, J7 PAD, J8 PAD, J9 PAD, U1 AMBIQ-APOLLO3KBR, Y1 32MHz

Commit message: Add C9 pad. Add FP for Artemis module.
Parts:
- removed J33: PAD, Module-Pads:PAD
- added J44, J45, J47, J48, J49: PAD.4X.6, Module-Pads:PAD.4X.6
- added J46: PAD.35X.35, Module-Pads:PAD.35X.35
- added LOGO1: SFE_LOGO_FLAME.05_INCH_INTERNAL, SparkFun-Aesthetics:SFE_LOGO_FLAME.05_INCH_INTERNAL
- added LOGO2: OSHW-LOGOS, SparkFun-Aesthetics:OSHW-LOGOS
- J1, J10, J11, J12, J13, J14, J15, J16, J17, J18, J19, J2, J20, J21, J22, J23, J24, J25, J26, J27, J28, J29, J3, J30, J31, J32, J34, J35, J36, J37, J38, J39, J4, J40, J41, J42, J43, J5, J6, J7, J8, J9: value PAD -> PAD.4X.6; device Module-Pads:PAD -> Module-Pads:PAD.4X.6
Connections:
- net GPIO33/SWO renamed ~AD33/SWO
- net MOSI renamed D7
- net MOSI3 renamed D38
- net RXI-1 renamed ~D25
- net SCL renamed ~D39
- net SDA renamed D40
- net TXO-1 renamed ~D24
- net ~AD31/RTS renamed ~AD31
- net ~D10/CTS renamed ~D26
- net ~MISO renamed ~D6
- net ~SCK renamed ~D5
- net ~SCL3/SCK3 renamed ~D42
- net ~SDA3/MISO3 renamed ~D43
- new net D9: J46.1, U1.GPIO9
- net GND: now also J44.1, J45.1, J47.1, J48.1; no longer J33.1
- net VDD: now also J49.1
Other:
- note added: "A/P"
- note added: "A/P/I2S"
- note added: "A/P/I2SDAT"
- note added: "A/P/PDMDATA"
- note added: "A/P/SCIO"
- note added: "Board thickness: 0.8mm"
- note added: "Distance between Layer 1/2: 0.14mm"
- note added: "Er: 4.58"
- note added: "MOSI0/CLKOUT"
- note added: "MOSI1/TX1/PDMCLK"
- note added: "MOSI3/RX1"
- note added: "Microstrip Calculation:"
- note added: "N. Seidle"
- note added: "P/A/RTS1/SCCLK"
- note added: "P/A/SDA3/MISO3/RX1"
- note added: "P/A/SWO"
- note added: "P/CTS1/SCRST"
- note added: "P/MOSI2/I2SWCLK"
- note added: "P/MOSI4"
- note added: "P/MOSI5/RX1/32kHz"
- note added: "P/PDMCLK"
- note added: "P/PDMCLK/SCCIO"
- note added: "P/RX1"
- note added: "P/SCL0/SCK0"
- note added: "P/SCL2/SCK2"
- note added: "P/SCL3/SCK3/TX1"
- note added: "P/SCL4/SCK4/TX1"
- note added: "P/SCL5/SCK5/TX0"
- note added: "P/SDA0/MISO0/I2SDAT"
- note added: "P/SDA2/MISO2/RX1"
- note added: "P/SDA5/MISO5/RX0"
- note added: "P/TX1/32kHz"
- note added: "Polygon Isolation: 5mil/0.127mm"
- note added: "RF Trace Width: 9.45mil/0.24mm"
- note added: "RX1/PDMDATA"
- note added: "SCL1/SCK1/TX1/SCCLK"
- note added: "SDA1/MISO1/RX1/SCCIO"
- note added: "SDA4/MISO4/RX1"
- note added: "https://chemandy.com/calculators/coplanar-waveguide-with-ground-calculator.htm"
- note removed: "External pullup on reset required"
- note removed: "Let's move the caps for DTR/GP14 reset combo off the module"
- note removed: "Pull up/down on JTAG SWIO removed"
- note removed: "UART0 is for programming"
- note removed: "nRF has 46 GPIO"
