File: Hardware/SparkFun_Artemis.sch (EAGLE design)
At the start: 87 parts, among them J1 PAD.4X.6, J10 PAD.4X.6, J11 PAD.4X.6, J12 PAD.4X.6, J13 PAD.4X.6, J14 PAD.4X.6, J15 PAD.4X.6, J16 PAD.4X.6, J17 PAD.4X.6, J18 PAD.4X.6, J19 PAD.4X.6, J2 PAD.4X.6, J20 PAD.4X.6, J21 PAD.4X.6, J22 PAD.35X.35, J23 PAD.4X.6, J24 PAD.4X.6, J25 PAD.4X.6, J26 PAD.4X.6, J27 PAD.4X.6, J28 PAD.4X.6, J29 PAD.4X.6, J3 PAD.4X.6, J30 PAD.4X.6, J31 PAD.4X.6, J32 PAD.4X.6, J33 PAD.4X.6, J34 PAD.4X.6, J35 PAD.4X.6, J36 PAD.4X.6, J37 PAD.4X.6, J38 PAD.35X.35, J39 PAD.4X.6, J4 PAD.4X.6, J40 PAD.4X.6, J41 PAD.4X.6, J42 PAD.4X.6, J43 PAD.4X.6, J44 PAD.4X.6, J45 PAD.4X.6, J46 PAD.4X.6, J47 PAD.4X.6, J48 PAD.4X.6, J49 PAD.4X.6, J5 PAD.4X.6, J50 PAD.4X.6, J51 PAD.4X.6, J52 PAD.4X.6, J53 PAD.4X.6, J54 PAD.4X.6, J55 PAD.4X.6, J56 PAD.4X.6, J57 PAD.4X.6, J58 PAD.4X.6, J59 PAD.4X.6, J6 PAD.4X.6, J7 PAD.4X.6, J8 PAD.4X.6, J9 PAD.4X.6, U1 AMBIQ-APOLLO3KBR, Y1 32MHz

Commit message: Adding new v1 FP of Artemis module
Connections:
- net D16 renamed AD16
- net D18 renamed ~D18
- net D19 renamed ~D19
- net D23 renamed ~D23
- net D34 renamed AD34
- net D45 renamed ~D45
Other:
- note added: "A/CMPIN0"
- note added: "A/CMPRF2"
- note added: "ADCD1N"
- note added: "ADCD1P"
- note added: "BLEIF_IRA/SWO"
- note added: "CMPRF1"
- note added: "P/CMPIN1"
- note added: "P/CMPOUT"
- note added: "P/CMPRF0"
- note added: "P/SWO"
- note added: "SLMISO"
- note added: "SLMOSI/SLSDA"
- note added: "SLSCK/SLSCL/CLKOUT"
- note added: "SLnCE"
- moved on the sheet: J18, J20, J29, J31, J40, J41, J42, J43, J45, J46, J48, J49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

Commit message: Adding dimensions
Parts:
- L2: device SparkFun-Coils:1.0μH-0805_WIDE-1.0μH-1.4A-0.07OHM -> SparkFun-Coils:1.0μH-0805_WIDE-1.0μH-1.45A-0.106OHM-1.0MM_H
Changed lines of the file:
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@@
 <?xml version="1.0" encoding="utf-8"?>
 <!DOCTYPE eagle SYSTEM "eagle.dtd">
-<eagle version="9.3.0">
+<eagle version="9.4.0">
 <drawing>
 <settings>
@@
 <layer number="115" name="ReferenceISLANDS" color="7" fill="1" visible="no" active="no"/>
 <layer number="116" name="Patch_BOT" color="9" fill="4" visible="no" active="no"/>
+<layer number="117" name="PM_Ref" color="26" fill="1" visible="yes" active="yes"/>
 <layer number="118" name="Rect_Pads" color="7" fill="1" visible="no" active="no"/>
+<layer number="119" name="PF_Ref" color="31" fill="1" visible="yes" active="yes"/>
+<layer number="120" name="WFL_Ref" color="25" fill="1" visible="yes" active="yes"/>
 <layer number="121" name="_tsilk" color="7" fill="1" visible="no" active="no"/>
 <layer number="122" name="_bsilk" color="7" fill="1" visible="no" active="no"/>
@@
 <part name="GND5" library="SparkFun-PowerSymbols" deviceset="GND" device=""/>
 <part name="L1" library="SparkFun-Coils" deviceset="2.2μH" device="-0805_WIDE-2.2μH-1.7A-0.14OHM" value="2.2μH"/>
-<part name="L2" library="SparkFun-Coils" deviceset="1.0μH" device="-0805_WIDE-1.0μH-1.4A-0.07OHM" value="1.0μH"/>
+<part name="L2" library="SparkFun-Coils" deviceset="1.0μH" device="-0805_WIDE-1.0μH-1.45A-0.106OHM-1.0MM_H" value="1.0μH"/>
 <part name="GND3" library="SparkFun-PowerSymbols" deviceset="GND" device=""/>
 <part name="C2" library="SparkFun-Capacitors" deviceset="4.7UF" device="-0402_TIGHT-6.3V-20%-X5R" value="4.7uF"/>
